File: schematics/circuit/htpm_control_display/htpm_control_display.kicad_pcb (KiCad board)
At the start: 2 copper layers, 0 parts

Commit message: Created HTPm CONTROL module display PCB.
Parts:
- added D1: RED, LED_THT:LED_D5.0mm, F.Cu at (142.2, 83.8)
- added D10: BLUE, LED_THT:LED_D5.0mm, F.Cu at (177.8, 88.9)
- added D11: BLUE, LED_THT:LED_D5.0mm, F.Cu at (154.9, 106.7)
- added D12: BLUE, LED_THT:LED_D5.0mm, F.Cu at (162.6, 106.7)
- added D13: BLUE, LED_THT:LED_D5.0mm, F.Cu at (170.2, 106.7)
- added D14: BLUE, LED_THT:LED_D5.0mm, F.Cu at (177.8, 106.7)
- added D15: BLUE, LED_THT:LED_D5.0mm, F.Cu at (154.9, 111.8)
- added D16: BLUE, LED_THT:LED_D5.0mm, F.Cu at (162.6, 111.8)
- added D17: BLUE, LED_THT:LED_D5.0mm, F.Cu at (170.2, 111.8)
- added D18: BLUE, LED_THT:LED_D5.0mm, F.Cu at (177.8, 111.8)
- added D2: RED, LED_THT:LED_D5.0mm, F.Cu at (142.2, 106.7)
- added D3: BLUE, LED_THT:LED_D5.0mm, F.Cu at (154.9, 83.8)
- added D4: BLUE, LED_THT:LED_D5.0mm, F.Cu at (162.6, 83.8)
- added D5: BLUE, LED_THT:LED_D5.0mm, F.Cu at (170.2, 83.8)
- added D6: BLUE, LED_THT:LED_D5.0mm, F.Cu at (177.8, 83.8)
- added D7: BLUE, LED_THT:LED_D5.0mm, F.Cu at (154.9, 88.9)
- added D8: BLUE, LED_THT:LED_D5.0mm, F.Cu at (162.6, 88.9)
- added D9: BLUE, LED_THT:LED_D5.0mm, F.Cu at (170.2, 88.9)
- added J1: Conn_01x10_Socket, Connector_PinHeader_2.00mm:PinHeader_1x10_P2.00mm_Vertical, F.Cu at (132.1, 76.2)
- added J2: Conn_01x10_Socket, Connector_PinHeader_2.00mm:PinHeader_1x10_P2.00mm_Vertical, F.Cu at (132.1, 119.4)
- added JP1: SolderJumper_2_Bridged, Jumper:SolderJumper-2_P1.3mm_Open_TrianglePad1.0x1.5mm, B.Cu at (154.9, 78.0)
- added JP10: SolderJumper_2_Bridged, Jumper:SolderJumper-2_P1.3mm_Open_TrianglePad1.0x1.5mm, B.Cu at (162.6, 100.9)
- added JP11: SolderJumper_2_Bridged, Jumper:SolderJumper-2_P1.3mm_Open_TrianglePad1.0x1.5mm, B.Cu at (170.2, 100.9)
- added JP12: SolderJumper_2_Bridged, Jumper:SolderJumper-2_P1.3mm_Open_TrianglePad1.0x1.5mm, B.Cu at (177.8, 100.9)
- added JP13: SolderJumper_2_Bridged, Jumper:SolderJumper-2_P1.3mm_Open_TrianglePad1.0x1.5mm, B.Cu at (154.9, 117.6)
- added JP14: SolderJumper_2_Bridged, Jumper:SolderJumper-2_P1.3mm_Open_TrianglePad1.0x1.5mm, B.Cu at (162.6, 117.6)
- added JP15: SolderJumper_2_Bridged, Jumper:SolderJumper-2_P1.3mm_Open_TrianglePad1.0x1.5mm, B.Cu at (170.2, 117.6)
- added JP16: SolderJumper_2_Bridged, Jumper:SolderJumper-2_P1.3mm_Open_TrianglePad1.0x1.5mm, B.Cu at (177.8, 117.6)
- added JP17: SolderJumper_2_Bridged, Jumper:SolderJumper-2_P1.3mm_Open_TrianglePad1.0x1.5mm, B.Cu at (114.3, 97.2)
- added JP18: SolderJumper_2_Bridged, Jumper:SolderJumper-2_P1.3mm_Open_TrianglePad1.0x1.5mm, B.Cu at (116.8, 97.2)
- added JP19: SolderJumper_2_Bridged, Jumper:SolderJumper-2_P1.3mm_Open_TrianglePad1.0x1.5mm, B.Cu at (119.4, 97.2)
- added JP2: SolderJumper_2_Bridged, Jumper:SolderJumper-2_P1.3mm_Open_TrianglePad1.0x1.5mm, B.Cu at (162.6, 78.0)
- added JP20: SolderJumper_2_Bridged, Jumper:SolderJumper-2_P1.3mm_Open_TrianglePad1.0x1.5mm, B.Cu at (121.9, 97.2)
- added JP21: SolderJumper_2_Bridged, Jumper:SolderJumper-2_P1.3mm_Open_TrianglePad1.0x1.5mm, B.Cu at (124.5, 97.2)
- added JP22: SolderJumper_2_Bridged, Jumper:SolderJumper-2_P1.3mm_Open_TrianglePad1.0x1.5mm, B.Cu at (127.0, 97.2)
- added JP23: SolderJumper_2_Bridged, Jumper:SolderJumper-2_P1.3mm_Open_TrianglePad1.0x1.5mm, B.Cu at (129.5, 97.2)
- added JP24: SolderJumper_2_Bridged, Jumper:SolderJumper-2_P1.3mm_Open_TrianglePad1.0x1.5mm, B.Cu at (132.1, 97.2)
- added JP25: SolderJumper_2_Bridged, Jumper:SolderJumper-2_P1.3mm_Open_TrianglePad1.0x1.5mm, B.Cu at (132.1, 86.4)
- added JP26: SolderJumper_2_Bridged, Jumper:SolderJumper-2_P1.3mm_Open_TrianglePad1.0x1.5mm, B.Cu at (129.5, 86.4)
- added JP27: SolderJumper_2_Bridged, Jumper:SolderJumper-2_P1.3mm_Open_TrianglePad1.0x1.5mm, B.Cu at (127.0, 86.4)
- added JP28: SolderJumper_2_Bridged, Jumper:SolderJumper-2_P1.3mm_Open_TrianglePad1.0x1.5mm, B.Cu at (124.5, 86.4)
- added JP29: SolderJumper_2_Bridged, Jumper:SolderJumper-2_P1.3mm_Open_TrianglePad1.0x1.5mm, B.Cu at (121.9, 86.4)
- added JP3: SolderJumper_2_Bridged, Jumper:SolderJumper-2_P1.3mm_Open_TrianglePad1.0x1.5mm, B.Cu at (170.2, 78.0)
- added JP30: SolderJumper_2_Bridged, Jumper:SolderJumper-2_P1.3mm_Open_TrianglePad1.0x1.5mm, B.Cu at (119.4, 86.4)
- added JP31: SolderJumper_2_Bridged, Jumper:SolderJumper-2_P1.3mm_Open_TrianglePad1.0x1.5mm, B.Cu at (116.8, 86.4)
- added JP32: SolderJumper_2_Bridged, Jumper:SolderJumper-2_P1.3mm_Open_TrianglePad1.0x1.5mm, B.Cu at (114.3, 86.4)
- added JP4: SolderJumper_2_Bridged, Jumper:SolderJumper-2_P1.3mm_Open_TrianglePad1.0x1.5mm, B.Cu at (177.8, 78.0)
- added JP5: SolderJumper_2_Bridged, Jumper:SolderJumper-2_P1.3mm_Open_TrianglePad1.0x1.5mm, B.Cu at (154.9, 94.7)
- added JP6: SolderJumper_2_Bridged, Jumper:SolderJumper-2_P1.3mm_Open_TrianglePad1.0x1.5mm, B.Cu at (162.6, 94.7)
- added JP7: SolderJumper_2_Bridged, Jumper:SolderJumper-2_P1.3mm_Open_TrianglePad1.0x1.5mm, B.Cu at (170.2, 94.7)
- added JP8: SolderJumper_2_Bridged, Jumper:SolderJumper-2_P1.3mm_Open_TrianglePad1.0x1.5mm, B.Cu at (177.8, 94.7)
- added JP9: SolderJumper_2_Bridged, Jumper:SolderJumper-2_P1.3mm_Open_TrianglePad1.0x1.5mm, B.Cu at (154.9, 100.9)
- added R1: 400Ω, Resistor_THT:R_Axial_DIN0204_L3.6mm_D1.6mm_P7.62mm_Horizontal, F.Cu at (127.0, 81.3)
- added R2: 400Ω, Resistor_THT:R_Axial_DIN0204_L3.6mm_D1.6mm_P7.62mm_Horizontal, F.Cu at (127.0, 104.1)
- added R3: 400Ω, Resistor_THT:R_Axial_DIN0204_L3.6mm_D1.6mm_P7.62mm_Horizontal, F.Cu at (141.0, 99.1)
- added R4: 400Ω, Resistor_THT:R_Axial_DIN0204_L3.6mm_D1.6mm_P7.62mm_Horizontal, F.Cu at (141.0, 94.0)
Routing:
- net GND: track 0.00 -> 179.9 mm
- net Net-(JP1-B): track 0.00 -> 76.3 mm
- net Net-(JP10-B): track 0.00 -> 76.3 mm
- net +3.3V: track 0.00 -> 61.8 mm
- net Net-(J1-Pin_3): track 0.00 -> 55.9 mm, vias 0 -> 1
- net Net-(J1-Pin_4): track 0.00 -> 55.5 mm, vias 0 -> 1
- net Net-(J1-Pin_5): track 0.00 -> 55.0 mm, vias 0 -> 1
- net Net-(J1-Pin_7): track 0.00 -> 54.7 mm, vias 0 -> 1
- net Net-(J1-Pin_6): track 0.00 -> 54.6 mm, vias 0 -> 1
- net Net-(J1-Pin_8): track 0.00 -> 53.7 mm, vias 0 -> 1
- net Net-(J1-Pin_9): track 0.00 -> 53.2 mm, vias 0 -> 1
- net Net-(J1-Pin_10): track 0.00 -> 52.8 mm, vias 0 -> 1
- net Net-(JP17-B): track 0.00 -> 24.0 mm
- net Net-(JP25-B): track 0.00 -> 22.1 mm
- net Net-(D2-A): track 0.00 -> 7.62 mm
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Other:
- board outline added: 73.7 x 48.3 mm

Commit message: Created HTPm CONTROL module display Gerbers.
Parts:
- added H1: MountingHole, MountingHole:MountingHole_2.5mm, F.Cu at (137.2, 88.9)
- added H2: MountingHole, MountingHole:MountingHole_2.5mm, F.Cu at (144.8, 116.8)
Other:
- board text added: "HTP!m CONTROL Module Display"
Changed lines of the file:
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@@
       (plot_on_all_layers_selection 0x0000000_00000000)
       (disableapertmacros false)
-      (usegerberextensions false)
+      (usegerberextensions true)
       (usegerberattributes true)
       (usegerberadvancedattributes true)
@@
       (outputformat 1)
       (mirror false)
-      (drillshape 1)
+      (drillshape 0)
       (scaleselection 1)
-      (outputdirectory "")
+      (outputdirectory "gerbers/")
     )
   )
@@
     )
   )
+  (footprint "MountingHole:MountingHole_2.5mm" (layer "F.Cu")
+    (at 144.78 116.84)
+    (descr "Mounting Hole 2.5mm, no annular")
+    (tags "mounting hole 2.5mm no annular")
+    (property "Sheetfile" "htpm_control_display.kicad_sch")
+    (property "Sheetname" "")
+    (property "ki_description" "Mounting Hole without connection")
+    (property "ki_keywords" "mounting hole")
+    (attr exclude_from_pos_files)
+    (fp_text reference "H2" (at 0 -3.5) (layer "F.SilkS")
+        (effects (font (size 1 1) (thickness 0.15)))
+    )
+    (fp_text value "MountingHole" (at 0 3.5) (layer "F.Fab")
+        (effects (font (size 1 1) (thickness 0.15)))
+    )
+    (fp_text user "${REFERENCE}" (at 0 0) (layer "F.Fab")
+        (effects (font (size 1 1) (thickness 0.15)))
+    )
+    (fp_circle (center 0 0) (end 2.5 0)
+      (stroke (width 0.15) (type solid)) (fill none) (layer "Cmts.User"))
+    (fp_circle (center 0 0) (end 2.75 0)
+      (stroke (width 0.05) (type solid)) (fill none) (layer "F.CrtYd"))
+    (pad "" np_thru_hole circle (at 0 0) (size 2.5 2.5) (drill 2.5) (layers "*.Cu" "*.Mask"))
+  )
   (footprint "Resistor_THT:R_Axial_DIN0204_L3.6mm_D1.6mm_P7.62mm_Horizontal" (layer "F.Cu")
     (at 140.97 99.06)
@@
     )
   )
+  (footprint "MountingHole:MountingHole_2.5mm" (layer "F.Cu")
+    (at 137.16 88.9)
+    (descr "Mounting Hole 2.5mm, no annular")
+    (tags "mounting hole 2.5mm no annular")
+    (property "Sheetfile" "htpm_control_display.kicad_sch")
+    (property "Sheetname" "")
+    (property "ki_description" "Mounting Hole without connection")
+    (property "ki_keywords" "mounting hole")
+    (attr exclude_from_pos_files)
+    (fp_text reference "H1" (at 0 -3.5) (layer "F.SilkS")
+        (effects (font (size 1 1) (thickness 0.15)))
+    )
+    (fp_text value "MountingHole" (at 0 3.5) (layer "F.Fab")
+        (effects (font (size 1 1) (thickness 0.15)))
+    )
+    (fp_text user "${REFERENCE}" (at 0 0) (layer "F.Fab")
+        (effects (font (size 1 1) (thickness 0.15)))
+    )
+    (fp_circle (center 0 0) (end 2.5 0)
+      (stroke (width 0.15) (type solid)) (fill none) (layer "Cmts.User"))
+    (fp_circle (center 0 0) (end 2.75 0)
+      (stroke (width 0.05) (type solid)) (fill none) (layer "F.CrtYd"))
+    (pad "" np_thru_hole circle (at 0 0) (size 2.5 2.5) (drill 2.5) (layers "*.Cu" "*.Mask"))
+  )
   (footprint "LED_THT:LED_D5.0mm" (layer "F.Cu")
     (at 154.94 106.68 90)
@@
   (gr_rect (start 111.76 73.66) (end 185.42 121.92)
     (stroke (width 0.1) (type default)) (fill none) (layer "Edge.Cuts"))
+  (gr_text "HTP!m CONTROL Module Display" (at 114.3 114.3 180) (layer "B.Cu")
+    (effects (font (size 1.5 1.5) (thickness 0.3) bold) (justify left bottom mirror))
+  )
   (segment (start 154.94 106.68) (end 152.4 104.14) (width 0.25) (layer "F.Cu") (net 1))
   (segment (start 139.7 83.82) (end 142.24 83.82) (width 0.25) (layer "F.Cu") (net 1))
