File: schematics/circuit/htpm_control_module_status/htpm_control_module_status.kicad_pcb (KiCad board)
At the start: 2 copper layers, 0 parts

Commit message: Created HTPm CONTROL Module Status PCB.
Parts:
- added D1: LED, LED_THT:LED_D5.0mm, F.Cu at (111.8, 78.7)
- added D10: LED, LED_THT:LED_D5.0mm, F.Cu at (119.4, 86.4)
- added D11: LED, LED_THT:LED_D5.0mm, F.Cu at (127.0, 86.4)
- added D12: LED, LED_THT:LED_D5.0mm, F.Cu at (134.6, 86.4)
- added D13: LED, LED_THT:LED_D5.0mm, F.Cu at (142.2, 86.4)
- added D14: LED, LED_THT:LED_D5.0mm, F.Cu at (149.9, 86.4)
- added D15: LED, LED_THT:LED_D5.0mm, F.Cu at (157.5, 86.4)
- added D16: LED, LED_THT:LED_D5.0mm, F.Cu at (165.1, 86.4)
- added D17: LED, LED_THT:LED_D5.0mm, F.Cu at (111.8, 101.6)
- added D18: LED, LED_THT:LED_D5.0mm, F.Cu at (119.4, 101.6)
- added D19: LED, LED_THT:LED_D5.0mm, F.Cu at (127.0, 101.6)
- added D2: LED, LED_THT:LED_D5.0mm, F.Cu at (119.4, 78.7)
- added D20: LED, LED_THT:LED_D5.0mm, F.Cu at (134.6, 101.6)
- added D21: LED, LED_THT:LED_D5.0mm, F.Cu at (142.2, 101.6)
- added D22: LED, LED_THT:LED_D5.0mm, F.Cu at (149.9, 101.6)
- added D23: LED, LED_THT:LED_D5.0mm, F.Cu at (157.5, 101.6)
- added D24: LED, LED_THT:LED_D5.0mm, F.Cu at (165.1, 101.6)
- added D25: LED, LED_THT:LED_D5.0mm, F.Cu at (111.8, 109.2)
- added D26: LED, LED_THT:LED_D5.0mm, F.Cu at (119.4, 109.2)
- added D27: LED, LED_THT:LED_D5.0mm, F.Cu at (127.0, 109.2)
- added D28: LED, LED_THT:LED_D5.0mm, F.Cu at (134.6, 109.2)
- added D29: LED, LED_THT:LED_D5.0mm, F.Cu at (142.2, 109.2)
- added D3: LED, LED_THT:LED_D5.0mm, F.Cu at (127.0, 78.7)
- added D30: LED, LED_THT:LED_D5.0mm, F.Cu at (149.9, 109.2)
- added D31: LED, LED_THT:LED_D5.0mm, F.Cu at (157.5, 109.2)
- added D32: LED, LED_THT:LED_D5.0mm, F.Cu at (165.1, 109.2)
- added D4: LED, LED_THT:LED_D5.0mm, F.Cu at (134.6, 78.7)
- added D5: LED, LED_THT:LED_D5.0mm, F.Cu at (142.2, 78.7)
- added D6: LED, LED_THT:LED_D5.0mm, F.Cu at (149.9, 78.7)
- added D7: LED, LED_THT:LED_D5.0mm, F.Cu at (157.5, 78.7)
- added D8: LED, LED_THT:LED_D5.0mm, F.Cu at (165.1, 78.7)
- added D9: LED, LED_THT:LED_D5.0mm, F.Cu at (111.8, 86.4)
- added H1: MountingHole, MountingHole:MountingHole_2.5mm, F.Cu at (106.7, 71.1)
- added H2: MountingHole, MountingHole:MountingHole_2.5mm, F.Cu at (172.7, 114.3)
- added J1: Conn_01x08_Socket, Connector_PinHeader_2.00mm:PinHeader_1x08_P2.00mm_Vertical, F.Cu at (142.6, 71.1)
- added J2: Conn_01x04_Socket, Connector_PinHeader_2.00mm:PinHeader_1x04_P2.00mm_Vertical, F.Cu at (172.7, 88.9)
- added J3: Conn_01x08_Socket, Connector_PinHeader_2.00mm:PinHeader_1x08_P2.00mm_Vertical, F.Cu at (142.6, 114.3)
Routing:
- net Net-(D16-A): track 0.00 -> 87.0 mm
- net Net-(D15-A): track 0.00 -> 75.8 mm
- net Net-(D1-A): track 0.00 -> 75.8 mm
- net Net-(D25-K): track 0.00 -> 70.8 mm
- net Net-(D1-K): track 0.00 -> 68.1 mm
- net Net-(D17-K): track 0.00 -> 65.2 mm
- net Net-(D10-A): track 0.00 -> 64.5 mm
- net Net-(D14-A): track 0.00 -> 64.5 mm
- net Net-(D10-K): track 0.00 -> 62.8 mm
- net Net-(D11-A): track 0.00 -> 54.5 mm
- net Net-(D13-A): track 0.00 -> 54.5 mm
- net Net-(D12-A): track 0.00 -> 51.6 mm
Other:
- board outline added: 71.1 x 48.3 mm
- board text added: "HTP!m CONTROL Module Status"
- board text added: "JLCJLCJLCJLC"
