File: schematics/circuit/htpm_control_numericals/htpm_control_numericals.kicad_pcb (KiCad board)
At the start: 2 copper layers, 99.1 x 99.1 mm, 28 parts, among them J1 Conn_01x05_Socket, U1 MAX7219, U10 D168K, U11 D168K, U12 D168K, U13 MAX7219, U14 D168K, U15 D168K, U16 D168K, U17 D168K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

Commit message: Created HTPm CONTROL Numericals PCB.
Parts:
- moved H2 109.3 mm to (109.2, 113.0)
- moved R3 26.8 mm to (171.4, 121.9)
- moved U11 26.8 mm to (168.9, 86.4)
- moved U15 26.8 mm to (168.9, 111.6)
- moved U17 26.8 mm to (143.5, 111.6)
- moved U18 26.8 mm to (161.3, 134.6)
- moved U5 26.8 mm to (153.7, 60.8)
- moved U6 26.8 mm to (168.9, 60.8)
- moved U9 26.8 mm to (143.5, 86.4)
- moved C2 26.8 mm to (127.7, 121.9)
- moved J1 26.8 mm to (98.3, 137.2)
- moved U1 26.8 mm to (110.5, 101.6)
- moved U3 26.8 mm to (125.7, 60.8)
- moved C3 26.8 mm to (168.4, 121.9)
- moved R2 26.8 mm to (130.8, 121.9)
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Routing:
- net GND: track 0.00 -> 197.1 mm, vias 0 -> 2
- net Net-(J1-Pin_3): track 0.00 -> 177.5 mm, vias 0 -> 4
- net Net-(J1-Pin_1): track 0.00 -> 167.7 mm
- net +5V: track 0.00 -> 149.5 mm, vias 0 -> 4
- net Net-(U1-SEG_G): track 0.00 -> 146.4 mm, vias 0 -> 6
- net Net-(U1-SEG_D): track 0.00 -> 144.3 mm, vias 0 -> 6
- net Net-(U1-SEG_E): track 0.00 -> 144.0 mm, vias 0 -> 6
- net Net-(U1-SEG_F): track 0.00 -> 135.0 mm, vias 0 -> 6
- net Net-(U1-SEG_C): track 0.00 -> 133.8 mm, vias 0 -> 7
- net Net-(U1-SEG_DP): track 0.00 -> 133.1 mm, vias 0 -> 7
- net Net-(U10-E): track 0.00 -> 132.1 mm, vias 0 -> 6
- net Net-(U10-G): track 0.00 -> 129.1 mm, vias 0 -> 10
- net Net-(U1-SEG_A): track 0.00 -> 127.9 mm, vias 0 -> 6
- net Net-(U1-SEG_B): track 0.00 -> 127.7 mm, vias 0 -> 7
- net Net-(U13-DIG_1): track 0.00 -> 126.7 mm
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
Commit message: Updated silkscreen on the HTPm CONTROL Numericals PCB.
Other:
- board text added: "HTP!m CONTROL Numericals by shawnd.xyz"
- board text added: "JLCJLCJLCJLC"
- board text added: "TARGET"
- board text added: "TIME"
- board text added: "VELOCITY"
Changed lines of the file:
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@@
     (property "ki_keywords" "mounting hole")
     (attr exclude_from_pos_files)
-    (fp_text reference "H2" (at 0 -3.5) (layer "F.SilkS")
-        (effects (font (size 1 1) (thickness 0.15)))
+    (fp_text reference "H2" (at 0 -3.5) (layer "B.SilkS")
+        (effects (font (size 1 1) (thickness 0.15)) (justify mirror))
     )
     (fp_text value "MountingHole" (at 0 3.5) (layer "F.Fab")
@@
     (property "ki_keywords" "mounting hole")
     (attr exclude_from_pos_files)
-    (fp_text reference "H1" (at 0 -3.5) (layer "F.SilkS")
-        (effects (font (size 1 1) (thickness 0.15)))
+    (fp_text reference "H1" (at 0 -3.5) (layer "B.SilkS")
+        (effects (font (size 1 1) (thickness 0.15)) (justify mirror))
     )
     (fp_text value "MountingHole" (at 0 3.5) (layer "F.Fab")
@@
     (property "ki_keywords" "R res resistor")
     (attr through_hole)
-    (fp_text reference "R2" (at 3.81 -1.92) (layer "F.SilkS")
-        (effects (font (size 1 1) (thickness 0.15)))
+    (fp_text reference "R2" (at 3.81 -1.92) (layer "B.SilkS")
+        (effects (font (size 1 1) (thickness 0.15)) (justify mirror))
     )
     (fp_text value "15kΩ" (at 3.81 1.92) (layer "F.Fab")
@@
     (property "ki_keywords" "R res resistor")
     (attr through_hole)
-    (fp_text reference "R3" (at 3.81 -1.92) (layer "F.SilkS")
-        (effects (font (size 1 1) (thickness 0.15)))
+    (fp_text reference "R3" (at 3.81 -1.92) (layer "B.SilkS")
+        (effects (font (size 1 1) (thickness 0.15)) (justify mirror))
     )
     (fp_text value "15kΩ" (at 3.81 1.92) (layer "F.Fab")
@@
     (property "ki_keywords" "LED 8-Digit Display Driver")
     (attr through_hole)
-    (fp_text reference "U13" (at 3.81 -2.33 90) (layer "F.SilkS")
-        (effects (font (size 1 1) (thickness 0.15)))
+    (fp_text reference "U13" (at 3.81 -2.33 90) (layer "B.SilkS")
+        (effects (font (size 1 1) (thickness 0.15)) (justify mirror))
     )
     (fp_text value "MAX7219" (at 3.81 30.27 90) (layer "F.Fab")
@@
     (property "ki_keywords" "LED 8-Digit Display Driver")
     (attr through_hole)
-    (fp_text reference "U1" (at 3.81 -2.33) (layer "F.SilkS")
-        (effects (font (size 1 1) (thickness 0.15)))
+    (fp_text reference "U1" (at 3.81 -2.33) (layer "B.SilkS")
+        (effects (font (size 1 1) (thickness 0.15)) (justify mirror))
     )
     (fp_text value "MAX7219" (at 3.81 30.27) (layer "F.Fab")
@@
     (property "ki_keywords" "R res resistor")
     (attr through_hole)
-    (fp_text reference "R1" (at 3.81 2.54 90) (layer "F.SilkS")
-        (effects (font (size 1 1) (thickness 0.15)))
+    (fp_text reference "R1" (at 3.81 2.54 90) (layer "B.SilkS")
+        (effects (font (size 1 1) (thickness 0.15)) (justify mirror))
     )
     (fp_text value "15kΩ" (at 3.81 1.92 90) (layer "F.Fab")
@@
     (property "ki_keywords" "LED 8-Digit Display Driver")
     (attr through_hole)
-    (fp_text reference "U18" (at 3.81 -2.33 90) (layer "F.SilkS")
-        (effects (font (size 1 1) (thickness 0.15)))
+    (fp_text reference "U18" (at 3.81 -2.33 90) (layer "B.SilkS")
+        (effects (font (size 1 1) (thickness 0.15)) (justify mirror))
     )
     (fp_text value "MAX7219" (at 3.81 30.27 90) (layer "F.Fab")
@@
     (property "ki_keywords" "connector")
     (attr through_hole)
-    (fp_text reference "J1" (at 0 -2.06 90) (layer "F.SilkS")
-        (effects (font (size 1 1) (thickness 0.15)))
+    (fp_text reference "J1" (at 0 -2.06 90) (layer "B.SilkS")
+        (effects (font (size 1 1) (thickness 0.15)) (justify mirror))
     )
     (fp_text value "Conn_01x05_Socket" (at 0 10.06 90) (layer "F.Fab") hide
@@
     (property "ki_keywords" "cap capacitor")
     (attr through_hole)
-    (fp_text reference "C2" (at 4.54 0) (layer "F.SilkS")
-        (effects (font (size 1 1) (thickness 0.15)))
+    (fp_text reference "C2" (at 4.54 0) (layer "B.SilkS")
+        (effects (font (size 1 1) (thickness 0.15)) (justify mirror))
     )
     (fp_text value "10μF" (at 1 3.25) (layer "F.Fab")
@@
     (property "ki_keywords" "cap capacitor")
     (attr through_hole)
-    (fp_text reference "C3" (at 4.54 0) (layer "F.SilkS")
-        (effects (font (size 1 1) (thickness 0.15)))
+    (fp_text reference "C3" (at 4.54 0) (layer "B.SilkS")
+        (effects (font (size 1 1) (thickness 0.15)) (justify mirror))
     )
     (fp_text value "10μF" (at 1 3.25) (layer "F.Fab")
@@
     (property "ki_keywords" "cap capacitor")
     (attr through_hole)
-    (fp_text reference "C1" (at 5.08 0 90) (layer "F.SilkS")
-        (effects (font (size 1 1) (thickness 0.15)))
+    (fp_text reference "C1" (at 5.08 0 -270) (layer "B.SilkS")
+        (effects (font (size 1 1) (thickness 0.15)) (justify mirror))
     )
     (fp_text value "10μF" (at 1 3.25 90) (layer "F.Fab")
@@
   (gr_rect (start 95.25 40.64) (end 194.31 139.7)
     (stroke (width 0.1) (type default)) (fill none) (layer "Edge.Cuts"))
+  (gr_text "JLCJLCJLCJLC" (at 123.19 74.93 90) (layer "B.SilkS")
+    (effects (font (size 1.5 1.5) (thickness 0.3) bold) (justify left bottom mirror))
+  )
+  (gr_text "HTP!m CONTROL Numericals\nby shawnd.xyz" (at 102.87 104.14 90) (layer "B.SilkS")
+    (effects (font (size 1.5 1.5) (thickness 0.3) bold) (justify left bottom mirror))
+  )
+  (gr_text "VELOCITY" (at 128.27 68.58 90) (layer "F.SilkS")
+    (effects (font (size 1.5 1.5) (thickness 0.3) bold) (justify right bottom))
+  )
+  (gr_text "TIME" (at 110.49 43.18 90) (layer "F.SilkS")
+    (effects (font (size 1.5 1.5) (thickness 0.3) bold) (justify right bottom))
+  )
+  (gr_text "TARGET" (at 128.27 93.98 90) (layer "F.SilkS")
+    (effects (font (size 1.5 1.5) (thickness 0.3) bold) (justify right bottom))
+  )
   (segment (start 165.83 124.46) (end 163.83 124.46) (width 0.25) (layer "F.Cu") (net 1))
   (segment (start 100.33 88.9) (end 102.87 88.9) (width 0.25) (layer "F.Cu") (net 1))
