File: schematics/circuit/htpm_control_module_display/htpm_control_module_display.kicad_pcb (KiCad board)
At the start: 2 copper layers, 73.7 x 43.2 mm, 58 parts, among them J1 Conn_01x10_Socket, J2 Conn_01x10_Socket

Commit message: Added user-facing text to HTPm CONTROL Module Display PCB.
Other:
- board text added: "MODULE"
- board text added: "OVER"
- board text added: "by shawnd.xyz"
Changed lines of the file:
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@@
     (effects (font (size 1.5 1.5) (thickness 0.3) bold) (justify left bottom mirror))
+  )
+  (gr_text "by shawnd.xyz" (at 177.8 78.74 90) (layer "B.SilkS")
+    (effects (font (size 1.5 1.5) (thickness 0.3) bold) (justify left mirror))
   )
   (gr_text "JLCJLCJLCJLC" (at 175.26 111.76) (layer "B.SilkS")
     (effects (font (size 1.5 1.5) (thickness 0.3) bold) (justify left bottom mirror))
   )
+  (gr_text "MODULE" (at 144.78 93.98) (layer "F.SilkS")
+    (effects (font (size 1.5 1.5) (thickness 0.3) bold) (justify left bottom))
+  )
+  (gr_text "OVER" (at 137.16 76.2) (layer "F.SilkS")
+    (effects (font (size 1.5 1.5) (thickness 0.3) bold) (justify bottom))
+  )
+  (gr_text "MODULE" (at 144.78 76.2) (layer "F.SilkS")
+    (effects (font (size 1.5 1.5) (thickness 0.3) bold) (justify left bottom))
+  )
+  (gr_text "OVER" (at 137.16 93.98) (layer "F.SilkS")
+    (effects (font (size 1.5 1.5) (thickness 0.3) bold) (justify bottom))
+  )
   (segment (start 170.18 104.14) (end 147.32 104.14) (width 0.25) (layer "B.Cu") (net 1))

Commit message: Updated recommended R and V values.
Parts:
- R1, R2, R3, R4: value 400Ω -> 10kΩ
Connections:
- J1 pad 1: +3.3V -> +5V
- J2 pad 1: +3.3V -> +5V
Changed lines of the file:
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@@
   (net 31 "Net-(JP25-B)")
   (net 32 "Net-(JP10-B)")
+  (net 33 "+5V")
   (footprint "LED_THT:LED_D5.0mm" (layer "F.Cu")
     (at 147.32 86.36 -90)
@@
       (stroke (width 0.1) (type solid)) (layer "F.Fab"))
     (pad "1" thru_hole rect (at 0 0 270) (size 1.35 1.35) (drill 0.8) (layers "*.Cu" "*.Mask")
-      (net 20 "+3.3V") (pinfunction "Pin_1") (pintype "passive"))
+      (net 33 "+5V") (pinfunction "Pin_1") (pintype "passive"))
     (pad "2" thru_hole oval (at 0 2 270) (size 1.35 1.35) (drill 0.8) (layers "*.Cu" "*.Mask")
       (net 1 "GND") (pinfunction "Pin_2") (pintype "passive"))
@@
         (effects (font (size 1 1) (thickness 0.15)) (justify mirror))
     )
-    (fp_text value "400Ω" (at 3.81 1.92) (layer "F.Fab")
+    (fp_text value "10kΩ" (at 3.81 1.92) (layer "F.Fab")
         (effects (font (size 1 1) (thickness 0.15)))
     )
@@
       (stroke (width 0.1) (type solid)) (layer "F.Fab"))
     (pad "1" thru_hole rect (at 0 0 270) (size 1.35 1.35) (drill 0.8) (layers "*.Cu" "*.Mask")
-      (net 20 "+3.3V") (pinfunction "Pin_1") (pintype "passive"))
+      (net 33 "+5V") (pinfunction "Pin_1") (pintype "passive"))
     (pad "2" thru_hole oval (at 0 2 270) (size 1.35 1.35) (drill 0.8) (layers "*.Cu" "*.Mask")
       (net 1 "GND") (pinfunction "Pin_2") (pintype "passive"))
@@
         (effects (font (size 1 1) (thickness 0.15)) (justify mirror))
     )
-    (fp_text value "400Ω" (at 3.81 1.92) (layer "F.Fab")
+    (fp_text value "10kΩ" (at 3.81 1.92) (layer "F.Fab")
         (effects (font (size 1 1) (thickness 0.15)))
     )
@@
         (effects (font (size 1 1) (thickness 0.15)) (justify mirror))
     )
-    (fp_text value "400Ω" (at 3.81 1.92) (layer "F.Fab")
+    (fp_text value "10kΩ" (at 3.81 1.92) (layer "F.Fab")
         (effects (font (size 1 1) (thickness 0.15)))
     )
@@
         (effects (font (size 1 1) (thickness 0.15)) (justify mirror))
     )
-    (fp_text value "400Ω" (at 3.81 1.92) (layer "F.Fab")
-        (effects (font (size 1 1) (thickness 0.15)))
-    )
+    (fp_text value "10kΩ" (at 3.81 1.92) (layer "F.Fab")
+        (effects (font (size 1 1) (thickness 0.15)))
+    )
