File: schematics/circuit/htpm_control_additional_info/htpm_control_additional_info.kicad_pcb (KiCad board)
At the start: 2 copper layers, 0 parts

Commit message: Created HTPm CONTROL Additional Info PCB.
Parts:
- added C1: 22μF, Capacitor_THT:CP_Radial_D4.0mm_P2.00mm, F.Cu at (207.5, 124.0)
- added C2: 22μF, Capacitor_THT:CP_Radial_D4.0mm_P2.00mm, F.Cu at (184.9, 124.0)
- added C3: 22μF, Capacitor_THT:CP_Radial_D4.0mm_P2.00mm, F.Cu at (143.0, 106.2)
- added C4: 22μF, Capacitor_THT:CP_Radial_D4.0mm_P2.00mm, F.Cu at (206.3, 50.5)
- added C5: 10μF, Capacitor_THT:CP_Radial_D4.0mm_P2.00mm, F.Cu at (134.4, 61.5)
- added C6: 10μF, Capacitor_THT:CP_Radial_D4.0mm_P2.00mm, F.Cu at (133.6, 88.1)
- added D1: RED, LED_THT:LED_D5.0mm, F.Cu at (152.4, 52.3)
- added D10: YELLOW, LED_THT:LED_D5.0mm, F.Cu at (167.6, 86.4)
- added D11: YELLOW, LED_THT:LED_D5.0mm, F.Cu at (160.0, 86.4)
- added D12: YELLOW, LED_THT:LED_D5.0mm, F.Cu at (152.4, 86.4)
- added D13: YELLOW, LED_THT:LED_D5.0mm, F.Cu at (205.7, 91.4)
- added D14: YELLOW, LED_THT:LED_D5.0mm, F.Cu at (198.1, 91.4)
- added D15: YELLOW, LED_THT:LED_D5.0mm, F.Cu at (190.5, 91.4)
- added D16: YELLOW, LED_THT:LED_D5.0mm, F.Cu at (182.9, 91.4)
- added D17: YELLOW, LED_THT:LED_D5.0mm, F.Cu at (175.3, 91.4)
- added D18: YELLOW, LED_THT:LED_D5.0mm, F.Cu at (167.6, 91.4)
- added D19: YELLOW, LED_THT:LED_D5.0mm, F.Cu at (160.0, 91.4)
- added D2: RED, LED_THT:LED_D5.0mm, F.Cu at (152.4, 59.9)
- added D20: YELLOW, LED_THT:LED_D5.0mm, F.Cu at (152.4, 91.4)
- added D3: GREEN, LED_THT:LED_D5.0mm, F.Cu at (152.4, 67.6)
- added D4: YELLOW, LED_THT:LED_D5.0mm, F.Cu at (152.4, 75.2)
- added D5: YELLOW, LED_THT:LED_D5.0mm, F.Cu at (205.7, 86.4)
- added D6: YELLOW, LED_THT:LED_D5.0mm, F.Cu at (198.1, 86.4)
- added D7: YELLOW, LED_THT:LED_D5.0mm, F.Cu at (190.5, 86.4)
- added D8: YELLOW, LED_THT:LED_D5.0mm, F.Cu at (182.9, 86.4)
- added D9: YELLOW, LED_THT:LED_D5.0mm, F.Cu at (175.3, 86.4)
- added H1: MountingHole, MountingHole:MountingHole_2.5mm, F.Cu at (182.9, 71.4)
- added H2: MountingHole, MountingHole:MountingHole_2.5mm, F.Cu at (156.5, 103.4)
- added J1: Conn_01x10_Socket, Connector_PinHeader_2.00mm:PinHeader_1x10_P2.00mm_Vertical, F.Cu at (138.2, 125.2)
- added J2: Conn_01x04_Socket, Connector_PinHeader_2.00mm:PinHeader_1x04_P2.00mm_Vertical, F.Cu at (114.3, 58.4)
- added J3: Conn_01x04_Socket, Connector_PinHeader_2.00mm:PinHeader_1x04_P2.00mm_Vertical, F.Cu at (114.3, 68.6)
- added J4: Conn_01x08_Socket, Connector_PinHeader_2.00mm:PinHeader_1x08_P2.00mm_Vertical, F.Cu at (114.3, 78.7)
- added J5: Conn_01x08_Socket, Connector_PinHeader_2.00mm:PinHeader_1x08_P2.00mm_Vertical, F.Cu at (114.3, 104.4)
- added J6: Conn_01x04_Socket, Connector_PinHeader_2.00mm:PinHeader_1x04_P2.00mm_Vertical, F.Cu at (114.3, 84.1)
- added J7: Conn_01x04_Socket, Connector_PinHeader_2.00mm:PinHeader_1x04_P2.00mm_Vertical, F.Cu at (114.3, 94.2)
- added J8: Conn_01x08_Socket, Connector_PinHeader_2.00mm:PinHeader_1x09_P2.00mm_Vertical, F.Cu at (130.3, 125.2)
- added J9: Conn_01x05_Socket, Connector_PinHeader_2.00mm:PinHeader_1x05_P2.00mm_Vertical, F.Cu at (114.8, 48.3)
- added R1: 680Ω, Resistor_THT:R_Axial_DIN0204_L3.6mm_D1.6mm_P7.62mm_Horizontal, F.Cu at (181.9, 54.9)
- added R10: 680Ω, Resistor_THT:R_Axial_DIN0204_L3.6mm_D1.6mm_P7.62mm_Horizontal, F.Cu at (172.2, 107.2)
- added R11: 680Ω, Resistor_THT:R_Axial_DIN0204_L3.6mm_D1.6mm_P7.62mm_Horizontal, F.Cu at (169.7, 107.2)
- added R12: 680Ω, Resistor_THT:R_Axial_DIN0204_L3.6mm_D1.6mm_P7.62mm_Horizontal, F.Cu at (167.1, 107.2)
- added R13: 680Ω, Resistor_THT:R_Axial_DIN0204_L3.6mm_D1.6mm_P7.62mm_Horizontal, F.Cu at (207.5, 107.2)
- added R14: 680Ω, Resistor_THT:R_Axial_DIN0204_L3.6mm_D1.6mm_P7.62mm_Horizontal, F.Cu at (205.0, 107.2)
- added R15: 680Ω, Resistor_THT:R_Axial_DIN0204_L3.6mm_D1.6mm_P7.62mm_Horizontal, F.Cu at (202.4, 107.2)
- added R16: 680Ω, Resistor_THT:R_Axial_DIN0204_L3.6mm_D1.6mm_P7.62mm_Horizontal, F.Cu at (199.9, 107.2)
- added R17: 680Ω, Resistor_THT:R_Axial_DIN0204_L3.6mm_D1.6mm_P7.62mm_Horizontal, F.Cu at (197.4, 107.2)
- added R18: 680Ω, Resistor_THT:R_Axial_DIN0204_L3.6mm_D1.6mm_P7.62mm_Horizontal, F.Cu at (194.8, 107.2)
- added R19: 680Ω, Resistor_THT:R_Axial_DIN0204_L3.6mm_D1.6mm_P7.62mm_Horizontal, F.Cu at (192.3, 107.2)
- added R2: 680Ω, Resistor_THT:R_Axial_DIN0204_L3.6mm_D1.6mm_P7.62mm_Horizontal, F.Cu at (181.9, 57.4)
- added R20: 680Ω, Resistor_THT:R_Axial_DIN0204_L3.6mm_D1.6mm_P7.62mm_Horizontal, F.Cu at (189.7, 107.2)
- added R21: 20kΩ, Resistor_THT:R_Axial_DIN0204_L3.6mm_D1.6mm_P7.62mm_Horizontal, F.Cu at (137.7, 64.0)
- added R22: 20kΩ, Resistor_THT:R_Axial_DIN0204_L3.6mm_D1.6mm_P7.62mm_Horizontal, F.Cu at (140.7, 103.6)
- added R3: 680Ω, Resistor_THT:R_Axial_DIN0204_L3.6mm_D1.6mm_P7.62mm_Horizontal, F.Cu at (181.9, 59.9)
- added R4: 680Ω, Resistor_THT:R_Axial_DIN0204_L3.6mm_D1.6mm_P7.62mm_Horizontal, F.Cu at (181.9, 62.5)
- added R5: 680Ω, Resistor_THT:R_Axial_DIN0204_L3.6mm_D1.6mm_P7.62mm_Horizontal, F.Cu at (184.9, 107.2)
- added R6: 680Ω, Resistor_THT:R_Axial_DIN0204_L3.6mm_D1.6mm_P7.62mm_Horizontal, F.Cu at (182.4, 107.2)
- added R7: 680Ω, Resistor_THT:R_Axial_DIN0204_L3.6mm_D1.6mm_P7.62mm_Horizontal, F.Cu at (179.8, 107.2)
- added R8: 680Ω, Resistor_THT:R_Axial_DIN0204_L3.6mm_D1.6mm_P7.62mm_Horizontal, F.Cu at (177.3, 107.2)
- added R9: 680Ω, Resistor_THT:R_Axial_DIN0204_L3.6mm_D1.6mm_P7.62mm_Horizontal, F.Cu at (174.8, 107.2)
- added U1: L7805, Package_TO_SOT_THT:TO-220-3_Horizontal_TabDown, F.Cu at (132.7, 117.1)
- added U2: 74HC595, Package_DIP:DIP-16_W7.62mm_Socket, F.Cu at (207.5, 111.3)
- added U3: 74HC595, Package_DIP:DIP-16_W7.62mm_Socket, F.Cu at (184.9, 111.3)
- added U4: 74HC595, Package_DIP:DIP-16_W7.62mm_Socket, F.Cu at (143.0, 118.9)
- added U5: 74HC595, Package_DIP:DIP-16_W7.62mm_Socket, F.Cu at (193.6, 50.5)
- added U6: MAX7219, Package_DIP:DIP-24_W7.62mm_Socket, F.Cu at (146.1, 67.1)
- added U7: MAX7219, Package_DIP:DIP-24_W7.62mm_Socket, F.Cu at (146.1, 92.7)
Routing:
- net GND: track 0.00 -> 458.7 mm, vias 0 -> 2
- net Net-(J1-Pin_1): track 0.00 -> 311.2 mm, vias 0 -> 3
- net Net-(J8-Pin_2): track 0.00 -> 156.6 mm, vias 0 -> 4
- net Net-(J8-Pin_1): track 0.00 -> 151.6 mm, vias 0 -> 4
- net Net-(J8-Pin_8): track 0.00 -> 123.7 mm, vias 0 -> 1
- net Net-(U4-QH'): track 0.00 -> 106.6 mm
- net Net-(J8-Pin_7): track 0.00 -> 94.0 mm, vias 0 -> 1
- net Net-(J8-Pin_6): track 0.00 -> 86.3 mm, vias 0 -> 1
- net Net-(J8-Pin_3): track 0.00 -> 83.9 mm, vias 0 -> 1
- net Net-(J8-Pin_9): track 0.00 -> 78.4 mm
- net Net-(D8-A): track 0.00 -> 50.4 mm
- net Net-(D12-A): track 0.00 -> 45.4 mm
- net Net-(D7-A): track 0.00 -> 41.4 mm
- net Net-(D20-A): track 0.00 -> 39.7 mm
- net Net-(D11-A): track 0.00 -> 36.3 mm
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Other:
- board outline added: 99.1 x 82 mm
- board text added: "0"
- board text added: "4"
- board text added: "ACCELERATE"
- board text added: "Controller"
- board text added: "DECELERATE"
- board text added: "DP"
- board text added: "EMERGENCY STOP"
- board text added: "HTP!m CONTROL Additional Info by shawnd.xyz"
- board text added: "JLCJLCJLCJLC"
- board text added: "Module Display"
- board text added: "Numericals"
- board text added: "OVERRIDE"
- board text added: "Status A"
- board text added: "Status B"

Commit message: Updated annotations.
Parts:
- moved J1 18.5 mm to (119.9, 128.3)
- moved C2 18.5 mm to (166.6, 127.0)
- moved C4 18.5 mm to (188.0, 53.6)
- moved C5 18.5 mm to (116.1, 64.5)
- moved D1 18.5 mm to (134.1, 55.4)
- moved D11 18.5 mm to (141.7, 89.4)
- moved D12 18.5 mm to (134.1, 89.4)
- moved D13 18.5 mm to (187.5, 94.5)
- moved D14 18.5 mm to (179.8, 94.5)
- moved D15 18.5 mm to (172.2, 94.5)
- moved D19 18.5 mm to (141.7, 94.5)
- moved D2 18.5 mm to (134.1, 63.0)
- moved D20 18.5 mm to (134.1, 94.5)
- moved D3 18.5 mm to (134.1, 70.6)
- moved D4 18.5 mm to (134.1, 78.2)
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