File: circuits/htpm_control/motherboard/motherboard.kicad_sch (KiCad schematic)
At the start: 55 parts, among them J5 Connector_Modcore, J6 Motor_Power, J7 Connector_Display, J8 Conn_01x40_Socket, J8 Connector_Motor_Driver, U1 74HC165, U5 74HC595, U7 L7805

Commit message: Created HTPm CONTROL Motherboard PCB.
Parts:
- removed H1, H2, H3, H4: MountingHole, MountingHole:MountingHole_2.5mm, symbol Mechanical:MountingHole
- R1, R10, R11, R12, R13, R14, R15, R16, R17, R18, R19, R2, R20, R21, R22, R23, R24, R25, R26, R27, R28, R29, R3, R30, R4, R5, R6, R7, R8, R9: value 10kΩ -> 4.7kΩ
Connections:
- net GND: now also J1.2 (GND), J4.1 (GND), J5.2 (GND), J7.6 (GND), J8.6 (GND), U7.2 (GND)
Other:
- company: (none) -> shawnd.xyz
- title: (none) -> HTP!m CONTROL Motherboard
